File: Silent_disco/amplifier.kicad_sch (KiCad schematic)
At the start: 0 parts

Commit message: add stuff
Parts:
- added U3: AD5664RBCPZ-3R2, CP_10_9_ADI, symbol AD5664RBCPZ-3R2:AD5664RBCPZ-3R2
- added U4: HT97180, symbol HT97180:HT97180
Changed lines of the file:
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@@
 	(generator_version "9.0")
 	(paper "A4")
+	(symbol
+		(lib_id "AD5664RBCPZ-3R2:AD5664RBCPZ-3R2")
+		(at 54.61 86.36 0)
+		(unit 1)
+		(exclude_from_sim no)
+		(in_bom yes)
+		(on_board yes)
+		(dnp no)
+		(fields_autoplaced yes)
+		(property "Reference" "U3"
+			(at 87.63 76.2 0)
+			(effects
+				(font
+					(size 1.524 1.524)
+				)
+			)
+		)
+		(property "Value" "AD5664RBCPZ-3R2"
+			(at 87.63 78.74 0)
+			(effects
+				(font
+					(size 1.524 1.524)
+				)
+			)
+		)
+		(property "Footprint" "CP_10_9_ADI"
+			(at 54.61 86.36 0)
+			(effects
+				(font
+					(size 1.27 1.27)
+					(italic yes)
+				)
+				(hide yes)
+			)
+		)
+		(property "Datasheet" "https://www.analog.com/media/en/technical-documentation/data-sheets/AD5624R_5644R_5664R.pdf"
+			(at 54.61 86.36 0)
+			(effects
+				(font
+					(size 1.27 1.27)
+					(italic yes)
+				)
+				(hide yes)
+			)
+		)
+		(property "Description" ""
+			(at 54.61 86.36 0)
+			(effects
+				(font
+					(size 1.27 1.27)
+				)
+				(hide yes)
+			)
+		)
+		(pin "4"
+		)
+		(pin "8"
+		)
+		(pin "11"
+		)
+		(pin "10"
+		)
+		(pin "5"
+		)
+		(pin "9"
+		)
+		(pin "2"
+		)
+		(pin "1"
+		)
+		(pin "6"
+		)
+		(pin "3"
+		)
+		(pin "7"
+		)
+		(instances
+			(project ""
+				(path "/4af49fe6-1b31-410d-a4f6-8a006077b266/89b335e4-deb8-44bf-bba8-15bcda0b3e9d"
+					(reference "U3")
+					(unit 1)
+				)
+			)
+		)
+	)
+	(symbol
+		(lib_id "HT97180:HT97180")
+		(at 176.53 99.06 0)
+		(unit 1)
+		(exclude_from_sim no)
+		(in_bom yes)
+		(on_board yes)
+		(dnp no)
+		(fields_autoplaced yes)
+		(property "Reference" "U4"
+			(at 191.77 87.5598 0)
+			(effects
+				(font
+					(size 1.27 1.27)
+				)
+			)
+		)
+		(property "Value" "HT97180"
+			(at 191.77 90.0998 0)
+			(effects
+				(font
+					(size 1.27 1.27)
+				)
+			)
+		)
+		(property "Footprint" ""
+			(at 176.53 82.55 0)
+			(effects
+				(font
+					(size 1.27 1.27)
+				)
+				(hide yes)
+			)
+		)
+		(property "Datasheet" ""
+			(at 176.53 82.55 0)
+			(effects
+				(font
+					(size 1.27 1.27)
+				)
+				(hide yes)
+			)
+		)
+		(property "Description" ""
+			(at 176.53 82.55 0)
+			(effects
+				(font
+					(size 1.27 1.27)
+				)
+				(hide yes)
+			)
+		)
+		(pin "13"
+		)
+		(pin "14"
+		)
+		(pin "11"
+		)
+		(pin ""
+		)
+		(pin "3"
+		)
+		(pin "10"
+		)
+		(pin "2"
+		)
+		(pin "16"
+		)
+		(pin "15"
+		)
+		(pin "1"
+		)
+		(pin "12"
+		)
+		(pin "5"
+		)
+		(pin "8"
+		)
+		(pin "4"
+		)
+		(pin "6"
+		)
+		(pin "7"
+		)
+		(instances
+			(project ""
+				(path "/4af49fe6-1b31-410d-a4f6-8a006077b266/89b335e4-deb8-44bf-bba8-15bcda0b3e9d"
+					(reference "U4")
+					(unit 1)
+				)
+			)
+		)
+	)
 )
