File: Silent_disco/esp32.kicad_sch (KiCad schematic)
At the start: 0 parts

Commit message: starting esp32 design
Parts:
- added C7, C9: C, symbol Device:C
- added C8: Sjekk datablad for value, symbol Device:C
- added R7: 10k, symbol Device:R
- added R8: 100, symbol Device:R
- added SW1, SW2: SW_Push, symbol Switch:SW_Push
- added U5: ESP32-WROOM-32E, RF_Module:ESP32-WROOM-32D, symbol RF_Module:ESP32-WROOM-32E
Connections:
- new net: R8.2, SW2.2
- new net +3.3V: C8.1, R7.2, U5.2 (VDD)
- new net BOOT: R8.1
- new net EN: C7.2, C9.1, R7.1, SW1.1, U5.3 (EN)
- new net GND: C7.1, C8.2, C9.2, SW1.2, SW2.1, U5.1 (GND), U5.15 (GND), U5.38 (GND), U5.39 (GND)
- new net TCK: U5.16 (IO13)
- new net TDI: U5.14 (IO12)
- new net TDO: U5.23 (IO15)
- new net TMS: U5.13 (IO14)

Commit message: Change ic charging ic
Parts:
- added C10: 100nF, symbol Device:C_Small
- added C11: 4.7uF, symbol Device:C_Small
- added C12: 22uF, symbol Device:C_Small
- added Q2: UMH3N, Package_TO_SOT_SMD:SOT-363_SC-70-6, symbol Transistor_BJT:UMH3N
- added TP1: TestPoint, symbol Connector:TestPoint
- added U7: CP2104, Package_DFN_QFN:QFN-24-1EP_4x4mm_P0.5mm_EP2.6x2.6mm, symbol Interface_USB:CP2104
Connections:
- net GND: now also C10.2, C11.2, C12.2
- new net: U7.2 (GND), U7.25 (GND)
- new net +5V: C10.1, C11.1, C12.1, U7.7 (REGIN), U7.8 (VBUS)
- new net D+: U7.3 (D+)
- new net D-: U7.4 (D-)
Other:
- moved on the sheet: C8, U5
