File: Silent_disco/power.kicad_sch (KiCad schematic)
At the start: 1 part, among them J1 USB_B_Micro

Commit message: husker ikke hva som ble endret her
Parts:
- added BT1: Battery_Cell, symbol Device:Battery_Cell
- added C1, C2: 1 μF, symbol Device:C
- added D1, D2, D3: LED, symbol Device:LED
- added Q1: PMOS, symbol Simulation_SPICE:PMOS
- added R1: 4k, symbol Device:R
- added R2, R3, R4: 470, symbol Device:R
- added R5: 10k, symbol Device:R
- added TH1: Thermistor_NTC, symbol Device:Thermistor_NTC
- added U1: MCP73833-FCI/UN, MSOP10_MC_MCH, symbol battery_MCP73833:MCP73833-FCI_UN
- added U2: TPS63001DRCR, DRC0010J, symbol TPS63001DRCR:TPS63001DRCR
Connections:
- net at J1.1 (VBUS): now also C2.2, D1.2 (A), D2.2 (A), D3.2 (A), Q1.2 (G), R5.2, U1.1 (VDD), U1.2 (VDD)
- net GND: now reaches J1.4 (ID)
- net GND: now also BT1.2 (-), C1.2, C2.1, R1.2, R5.1, TH1.2, U1.5 (VSS)
- new net: BT1.1 (+), C1.1, Q1.3 (S), U1.10 (VBAT), U1.9 (VBAT)
- new net: R1.1, U1.6 (PROG)
- new net: TH1.1, U1.8 (THERM)
- new net: R3.2, U1.3 (STAT1)
- new net: R2.2, U1.4 (STAT2)
- new net: R4.2, U1.7 (*PG)
- new net: D1.1 (K), R3.1
- new net: D2.1 (K), R2.1
- new net: D3.1 (K), R4.1
- new net LOAD: Q1.1 (D)
Other:
- moved on the sheet: J1

Commit message: add stuff
Parts:
- added C3, C5, C6: 10 μF, symbol Device:C
- added C4: 0.1μF, symbol Device:C
- added L1: 2.2μH, symbol Device:L
- added R6: 100, symbol Device:R
Connections:
- net GND: now also U2.3 (PGND), U2.9 (GND), C3.2, C4.2
- net LOAD: now also U2.1 (VOUT), U2.10 (FB), C5.1, C6.1; no longer Q1.1 (D)
- net at U2.2 (L2): now also L1.2
- net at U2.4 (L1): now also L1.1
- net at U2.5 (VIN): now also Q1.1 (D), C3.1, R6.2
- net at U2.6 (EN): now also U2.7 (PS_SYNC), U2.8 (VINA), C4.1, R6.1
Other:
- moved on the sheet: BT1, C1, Q1, U2

Commit message: starting esp32 design
Parts:
- removed J1: USB_B_Micro, symbol Connector:USB_B_Micro
- added J1: USB_C_Receptacle_USB2.0_16P, symbol Connector:USB_C_Receptacle_USB2.0_16P
- added R10, R9: 5.1k, symbol Device:R
Connections:
- net GND: now also C5.2, C6.2, J1.A1 (GND), J1.A12 (GND), J1.B1 (GND), J1.B12 (GND), J1.S1 (SHIELD), R10.1, R9.2
- net at C2.2, D1.2 (A), D2.2 (A)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: now also J1.A4 (VBUS), J1.A9 (VBUS), J1.B4 (VBUS), J1.B9 (VBUS)
- new net: J1.B5 (CC2), R10.2
- new net: J1.A5 (CC1), R9.1
- new net D+: J1.A6 (D+), J1.B6 (D+)
- new net D-: J1.A7 (D-), J1.B7 (D-)
- no-connect marks 0 -> 3
Other:
- moved on the sheet: C2

Commit message: Change ic charging ic
Parts:
- removed C1, C2: 1 μF, symbol Device:C
- removed D1, D2, D3: LED, symbol Device:LED
- removed Q1: PMOS, symbol Simulation_SPICE:PMOS
- removed R1: 4k, symbol Device:R
- removed R2, R3, R4: 470, symbol Device:R
- removed R5: 10k, symbol Device:R
- removed U1: MCP73833-FCI/UN, MSOP10_MC_MCH, symbol battery_MCP73833:MCP73833-FCI_UN
- added C1: 10uF, symbol Device:C_Small
- added C13, C2: 4.7uF, symbol Device:C_Small
- added F1: 1A polyfuse, symbol Device:Polyfuse_Small
- added FB1: BLM21PG221, symbol Device:FerriteBead_Small
- added U1, U8: MCP73871T-2CCI/ML, QFN20_4x4MC_MCH, symbol MCP73871T-2CCI-ML:MCP73871T-2CCI_ML
- added U6: USBLC6-2P6, Package_TO_SOT_SMD:SOT-666, symbol Power_Protection:USBLC6-2P6
Connections:
- net D+: now also U6.6 (I/O1); no longer J1.A6 (D+), J1.B6 (D+)
- net D-: now also U6.1 (I/O1); no longer J1.A7 (D-), J1.B7 (D-)
- net GND: now also C1.2, C13.2, C2.2, U1.10 (VSS), U1.11 (VSS), U6.2 (GND)
- net at C3.1, R6.2, U2.5 (VIN): now also C13.1, U8.1 (OUT), U8.20 (OUT)
- net +5VP: now reaches J1.A4 (VBUS), J1.A9 (VBUS), J1.B4 (VBUS), J1.B9 (VBUS)
- net +5VP: now also FB1.2
- net at BT1.1 (+): now also C2.1, U8.14 (VBAT), U8.15 (VBAT), U8.16 (VBAT_SENSE)
- net at TH1.1: now also U8.5 (THERM)
- new net: F1.2, FB1.1
- new net: J1.A6 (D+), J1.B6 (D+), U6.4 (I/O2)
- new net: J1.A7 (D-), J1.B7 (D-), U6.3 (I/O2)
- new net +5V: C1.1, F1.1, U6.5 (VBUS), U8.18 (IN), U8.19 (IN)
- no-connect marks 3 -> 2
Other:
- moved on the sheet: C3, C4, C5, C6, L1, R10, R6, R9, U2

Commit message: husker ikke hva jeg gjorde
Parts:
- added Q1: NPN, symbol Simulation_SPICE:NPN
- added R1: 4k, symbol Device:R_Small
- added R2: 15K, symbol Device:R_Small
Connections:
- net +5V: now also U8.4 (PROG2)
- net GND: now also U8.3 (SEL), R1.2, R2.2
- net LOAD: now also Q1.1 (C)
- net at U8.12 (PROG3): now also R2.1
- net at U8.13 (PROG1): now also R1.1
- net LBO: now reaches U8.8 (STAT1/*LBO)
- net LBO: now also Q1.2 (B)
- new net LBO_esp32: Q1.3 (E)
Other:
- moved on the sheet: C13
